Commit message: Added position sliders to GUI and created IK chain

File: robot.URDF (robot description, URDF)
Before this commit: robot robotarm, 6 links, 5 joints
Links:
- removed link bone_b
- removed link bone_c
- link bone_a: geometry 
Joints:
- removed joint elbow
- removed joint wrist
- joint floor: limit lower=0.0 upper=270.0 effort=0.0 velocity=0.0 -> (none)
- joint platform: limit lower=0.0 upper=0.0 effort=0.0 velocity=0.0 -> lower=0.0 upper=2.4783675 effort=0.0 velocity=0.0; origin xyz=0 0 10 rpy=0 0 0 -> xyz=0 0 10 rpy=0 3.1415926 0
